File: hardware/KiCAD/jpod-v1.0/jpod-v1.0.kicad_sch (KiCad schematic)
At the start: 70 parts, among them J1 SD_Card, J2 SPI_DEBUG, J3 LCD_HEADER, J4 3.5mm Jack, P1 BATTERY_CONN, Q1 AO3400A, U1 ESP32, U2 1.8V Regulator, U3 DAC, U4 Charger, U5 Buck Boost, U6 Fuel Gauge

Commit message: Implemented the UART bridge and power + ESD. Still needs some work on the transistors, but each bus should be connected now.
Parts:
- added C27, C31: 0.1uF, Capacitor_SMD:C_0603_1608Metric, symbol Device:C
- added C30: 4.7uF, Capacitor_SMD:C_0603_1608Metric, symbol Device:C
- added J5: USB_CON, jpod:USB4105-GF-A, symbol jpod:USB4105-GF-A
- added Q4, Q5: MMBT3904, Package_TO_SOT_SMD:SOT-23, symbol Transistor_BJT:MMBT3904
- added R24, R25: 5.1K, Resistor_SMD:R_0603_1608Metric, symbol Device:R
- added R26: 22.1K, Resistor_SMD:R_0603_1608Metric, symbol Device:R
- added R27: 47.5K, Resistor_SMD:R_0603_1608Metric, symbol Device:R
- added R28: 2K, Resistor_SMD:R_0603_1608Metric, symbol Device:R
- added R29, R30: 10K, Resistor_SMD:R_0603_1608Metric, symbol Device:R
- added U7: UART_Bridge, jpod:CP2102N-A02-GQFN24R, symbol jpod:CP2102N-A02-GQFN24R
- added U8: ESD, jpod:USBLC6-2P6, symbol jpod:USBLC6-2P6
- U2: value 1.8V Regulator -> 1.8V_Regulator
- U5: value Buck Boost -> Buck_Boost; DESCRIPTION High Efficiency Single Inductor Buck-Boost Converter with 4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 -> (none)
- U6: value Fuel Gauge -> Fuel_Gauge
Connections:
- net +3V3: now also C30.2, C31.2, R28.2, U7.5 (VIO), U7.6 (VDD), U7.7 (VREGIN)
- net GND: now also C27.1, C30.1, C31.1, J5.A1_B12 (GND), J5.B1_A12 (GND__1), J5.SH1 (SHELL_GND), J5.SH2 (SHELL_GND__1), J5.SH3 (SHELL_GND__2), J5.SH4 (SHELL_GND__3), R24.2, R25.1, R27.2, U7.2 (GND), U7.25 (GND__1), U8.2 (GND)
- net VBUS: now also C27.2, J5.A4_B9 (VBUS), J5.B4_A9 (VBUS__1), R26.2, U8.5 (VBUS)
- net RX: now reaches U1.34 (RXD0)
- net TX: now reaches U1.35 (TXD0)
- new net: J5.A5 (CC1), R24.1
- new net: Q4.2 (E), R30.1, U7.23 (~{DTR})
- new net: Q5.1 (B), R30.2
- new net: Q5.2 (E), R29.1, U7.19 (~{RTS})
- new net: R26.1, R27.1, U7.8 (VBUS)
- new net: Q4.1 (B), R29.2
- new net: R28.1, U7.9 (~{RST})
- new net: J5.B5 (CC2), R25.2
- new net D+: U8.6 (I/01)
- new net D-: U8.4 (I/02)
- new net DN: J5.A7 (DN1), J5.B7 (DN2), U8.3 (I/02)
- new net DP: J5.A6 (DP1), J5.B6 (DP2), U8.1 (I/01)
- new net ESP_EN: Q5.3 (C)
- new net ESP_IO0: Q4.3 (C)
- new net ESP_RXD0: U7.21 (TXD)
- new net ESP_TXD0: U7.20 (RXD)
- new net I/01: U7.3 (D+)
- new net I/02: U7.4 (D-)
- no-connect marks 12 -> 24
Other:
- note added: "1: Emitter (Source) 2: Base (Gate) 3: Collector (Drain)"
- note added: "References from ESP RX to UART TX"
- note added: "References from ESP TX to UART RX"
- moved on the sheet: C1, C10, C11, C12, C13, C14, C15, C16, C17, C18, C19, C2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
